File: eagle/MySLipo_v2.0.brd (EAGLE design)
At the start: 78 x 21 mm, 23 parts, among them IC1 ATMEGA328, U1 USB_CHARGER, U2 HT7333, U3 ATSHA204A

Commit message: v2.0
Parts:
- removed J$1: ANTENNATINY, WeMos-Lora:SMA_UFL_PAD_TINY
- removed JP1: (no value), pinhead:1X07
- removed R3, R4: 4K7, rcl:R0805
- removed R7: 10K, rcl:R0805
- removed RFM69W: RADIO_RFM69W_MIN_PAD, mysensors:RFM69W_MIN_PAD
- added C5, C6: 100n, rcl:C0805
- added LED1: yellow, mysensors:LED_0805
- added R10, R11: 10K, rcl:R0805
- added R12: 1K2, rcl:R0805
- added R8, R9: 1M, rcl:R0805
- added S1, S2: MEDER, moje:15X
- BATT1: value SINGLE_BATTERY_HOLDER18650 -> LI-PO_18650
- NRF24L01: value WIRELESS-NRF24L01SMD2 -> (none)
- NRF24L01+LNA+PA: value WIRELESS-NRF24L01-PA-EXTSMD -> (none)
- R5: value 120K -> 1M
- R6: value 220K -> 330K
- U2: device moje:SOT-89 -> my-power:SOT89
- moved U3 4.13 mm to (36.8, 18.4)
- moved C2 3.31 mm to (43.6, 17.8)
- moved NRF24L01+LNA+PA 3.24 mm to (46.4, 3.17)
- moved NRF24L01 3.19 mm to (53.0, 5.08)
- moved DS18B20 1.27 mm to (75.9, 17.2)
- moved R2 1.27 mm to (71.8, 18.4), turned to 90 degrees
- moved U2 0.32 mm to (30.2, 17.1)
- renumbered 18500 to BATT1
Connections:
- net N$5 renamed CE
- removed net A0: IC1.23, JP1.1, R7.1
- removed net A1: IC1.24, JP1.2
- removed net ANT: J$1.ANT1, J$1.ANT2, J$1.ANT3, RFM69W.10
- removed net N$6: IC1.14, NRF24L01+LNA+PA.6, NRF24L01.5, RFM69W.15
- removed net N$8: BATT1.+, U1.B+
- removed net SCL: IC1.28, JP1.4, R4.1
- removed net SDA: IC1.27, JP1.3, R3.1
- new net CSN: IC1.14, NRF24L01+LNA+PA.6, NRF24L01.5
- new net D3: IC1.1, R11.1
- new net D7: IC1.11, LED1.1
- new net N$17: LED1.2, R12.2
- new net N$2: C5.1, R10.2, R9.2, S1.P$1
- new net N$3: C6.2, R11.2, R8.1, S2.P$1
- net +3V3: now also C5.2, C6.1, R8.2, R9.1; no longer JP1.7, R3.2, R4.2, RFM69W.8
- net 1-WIRE_SUPPLY: now also DS18B20.S; no longer DS18B20.D
- net D2: now also IC1.32, R10.1; no longer IC1.1, JP1.5
- net GND: now also DS18B20.D, R12.1, S1.P$2, S2.P$2; no longer DS18B20.S, J$1.GND1, J$1.GND2, J$1.GND3, J$1.GND4, JP1.6, R7.2, RFM69W.11, RFM69W.9
- net MISO: no longer RFM69W.13
- net MOSI: no longer RFM69W.14
- net N$1: no longer IC1.32, RFM69W.2
- net SCK: no longer RFM69W.12
- net VBATT: now also BATT1.+, U1.B+
- net VCC: no longer U2.2@1
Routing:
- net D7: track 0.00 -> 41.4 mm, vias 0 -> 2
- net N$6: track 35.9 -> 0.00 mm, vias 1 -> 0
- net D3: track 0.00 -> 34.8 mm, vias 0 -> 2
- net GND: track 34.2 -> 0.00 mm, vias 14 -> 7
- net A0: track 30.1 -> 0.00 mm
- net D2: track 25.7 -> 55.1 mm, vias 1 -> 4
- net VBATT: track 49.9 -> 78.1 mm
- net N$1: track 35.9 -> 8.46 mm, vias 2 -> 0
- net SDA: track 26.9 -> 0.00 mm, vias 1 -> 0
- net SCL: track 26.0 -> 0.00 mm, vias 1 -> 0
- net A1: track 22.9 -> 0.00 mm
- net N$8: track 22.9 -> 0.00 mm
- net CSN: track 0.00 -> 19.9 mm, vias 0 -> 1
- net N$2: track 0.00 -> 17.8 mm
- net MOSI: track 40.1 -> 23.3 mm
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- removed copper zone on layer 1, net N$12
- removed copper zone on layer 1, net N$14
- removed copper zone on layer 1, net N$15
- removed copper zone on layer 1, net N$4
- removed copper zone on layer 1, net N$7
Other:
- board text added: "MySLipo v2.0"
- board text removed: "3V3"
- board text removed: "A0"
- board text removed: "A1"
- board text removed: "D2"
- board text removed: "GND"
- board text removed: "MySLipo v1.0"
- board text removed: "SCL"
- board text removed: "SDA"

Commit message: eagle update
Connections:
- new net +BATT: BATT1.+, U1.B+
- net VBATT: no longer BATT1.+, U1.B+
Routing:
- net VBATT: track 78.1 -> 49.9 mm
- net +BATT: track 0.00 -> 22.9 mm
Changed lines of the file:
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@@
 <?xml version="1.0" encoding="utf-8"?>
 <!DOCTYPE eagle SYSTEM "eagle.dtd">
-<eagle version="8.3.1">
+<eagle version="9.2.2">
 <drawing>
 <settings>
-<setting alwaysvectorfont="no"/>
+<setting alwaysvectorfont="yes"/>
 <setting keepoldvectorfont="yes"/>
 <setting verticaltext="up"/>
@@
 <wire x1="78" y1="21" x2="0" y2="21" width="0" layer="20"/>
 <wire x1="0" y1="21" x2="0" y2="0" width="0" layer="20"/>
-<text x="31.75" y="3.4925" size="0.9" layer="112" font="vector" ratio="15" align="bottom-center">V</text>
-<text x="29.21" y="3.4925" size="0.9" layer="112" font="vector" ratio="15" align="bottom-center">R</text>
-<text x="34.29" y="3.4925" size="0.9" layer="112" font="vector" ratio="15" align="bottom-center">G</text>
-<text x="36.83" y="3.4925" size="0.9" layer="112" font="vector" ratio="15" align="bottom-center">O</text>
-<text x="39.37" y="3.4925" size="0.9" layer="112" font="vector" ratio="15" align="bottom-center">C</text>
-<text x="41.91" y="3.4925" size="0.9" layer="112" font="vector" ratio="15" align="bottom-center">I</text>
+<text x="31.75" y="3.4925" size="0.9" layer="27" font="vector" ratio="15" align="bottom-center">V</text>
+<text x="29.21" y="3.4925" size="0.9" layer="27" font="vector" ratio="15" align="bottom-center">R</text>
+<text x="34.29" y="3.4925" size="0.9" layer="27" font="vector" ratio="15" align="bottom-center">G</text>
+<text x="36.83" y="3.4925" size="0.9" layer="27" font="vector" ratio="15" align="bottom-center">O</text>
+<text x="39.37" y="3.4925" size="0.9" layer="27" font="vector" ratio="15" align="bottom-center">C</text>
+<text x="41.91" y="3.4925" size="0.9" layer="27" font="vector" ratio="15" align="bottom-center">I</text>
 <text x="0.9525" y="1.27" size="0.9" layer="112" font="vector" ratio="18" align="center-left">MySLipo v2.0</text>
 <text x="12.3825" y="1.27" size="0.8" layer="112" font="vector" ratio="15" align="center-left">www.github.com/pilotak</text>
@@
 <param name="dpMaxLengthDifference" value="10mm"/>
 <param name="dpGapFactor" value="2.5"/>
-<param name="checkGrid" value="0"/>
 <param name="checkAngle" value="1"/>
 <param name="checkFont" value="1"/>
 <param name="checkRestrict" value="1"/>
+<param name="checkStop" value="0"/>
+<param name="checkValues" value="0"/>
+<param name="checkNames" value="1"/>
+<param name="checkWireStubs" value="1"/>
+<param name="checkPolygonWidth" value="0"/>
 <param name="useDiameter" value="13"/>
 <param name="maxErrors" value="50"/>
@@
 <attribute name="VALUE" x="21.59" y="18.57375" size="0.9" layer="27" font="vector" ratio="15" align="top-center"/>
 </element>
-<element name="S2" library="moje" package="15X" value="MEDER" x="55.5625" y="19.5"/>
-<element name="S1" library="moje" package="15X" value="MEDER" x="55.5625" y="1.5" rot="R180"/>
-<element name="R8" library="rcl" package="R0805" value="1M" x="49.53" y="17.145"/>
-<element name="R9" library="rcl" package="R0805" value="1M" x="75.565" y="6.985" rot="R180"/>
-<element name="C5" library="rcl" package="C0805" value="100n" x="75.565" y="4.1275"/>
-<element name="C6" library="rcl" package="C0805" value="100n" x="54.9275" y="17.145"/>
-<element name="R10" library="rcl" package="R0805" value="10K" x="75.565" y="1.27" rot="R180"/>
-<element name="R11" library="rcl" package="R0805" value="10K" x="60.325" y="17.145" rot="R180"/>
-<element name="LED1" library="mysensors" package="LED_0805" value="yellow" x="66.3575" y="18.415" rot="R90"/>
-<element name="R12" library="rcl" package="R0805" value="1K2" x="68.8975" y="18.415" rot="R90"/>
-<element name="U2" library="my-power" package="SOT89" value="HT7333" x="30.1625" y="17.145"/>
+<element name="S2" library="moje" package="15X" value="MEDER" x="55.5625" y="19.5" smashed="yes">
+<attribute name="NAME" x="50.4825" y="18.865" size="0.8128" layer="25"/>
+<attribute name="VALUE" x="56.8325" y="18.865" size="0.8128" layer="27"/>
+</element>
+<element name="S1" library="moje" package="15X" value="MEDER" x="55.5625" y="1.5" smashed="yes" rot="R180">
+<attribute name="NAME" x="60.6425" y="2.135" size="0.8128" layer="25" rot="R180"/>
+<attribute name="VALUE" x="54.2925" y="2.135" size="0.8128" layer="27" rot="R180"/>
+</element>
+<element name="R8" library="rcl" package="R0805" value="1M" x="49.53" y="17.145" smashed="yes">
+<attribute name="NAME" x="48.895" y="18.415" size="1.27" layer="25"/>
+<attribute name="VALUE" x="48.895" y="14.605" size="1.27" layer="27"/>
+</element>
+<element name="R9" library="rcl" package="R0805" value="1M" x="75.565" y="6.985" smashed="yes" rot="R180">
+<attribute name="NAME" x="76.2" y="5.715" size="1.27" layer="25" rot="R180"/>
+<attribute name="VALUE" x="76.2" y="9.525" size="1.27" layer="27" rot="R180"/>
+</element>
+<element name="C5" library="rcl" package="C0805" value="100n" x="75.565" y="4.1275" smashed="yes">
+<attribute name="NAME" x="74.295" y="5.3975" size="1.27" layer="25"/>
+<attribute name="VALUE" x="74.295" y="1.5875" size="1.27" layer="27"/>
+</element>
+<element name="C6" library="rcl" package="C0805" value="100n" x="54.9275" y="17.145" smashed="yes">
+<attribute name="NAME" x="53.6575" y="18.415" size="1.27" layer="25"/>
+<attribute name="VALUE" x="53.6575" y="14.605" size="1.27" layer="27"/>
+</element>
+<element name="R10" library="rcl" package="R0805" value="10K" x="75.565" y="1.27" smashed="yes" rot="R180">
+<attribute name="NAME" x="76.2" y="0" size="1.27" layer="25" rot="R180"/>
+<attribute name="VALUE" x="76.2" y="3.81" size="1.27" layer="27" rot="R180"/>
+</element>
+<element name="R11" library="rcl" package="R0805" value="10K" x="60.325" y="17.145" smashed="yes" rot="R180">
+<attribute name="NAME" x="60.96" y="15.875" size="1.27" layer="25" rot="R180"/>
+<attribute name="VALUE" x="60.96" y="19.685" size="1.27" layer="27" rot="R180"/>
+</element>
+<element name="LED1" library="mysensors" package="LED_0805" value="yellow" x="66.3575" y="18.415" smashed="yes" rot="R90">
+<attribute name="NAME" x="65.4825" y="17.542" size="0.8128" layer="25" ratio="15" rot="R90"/>
+<attribute name="VALUE" x="68.2575" y="17.415" size="0.762" layer="27" ratio="10" rot="R90"/>
+</element>
+<element name="R12" library="rcl" package="R0805" value="1K2" x="68.8975" y="18.415" smashed="yes" rot="R90">
+<attribute name="NAME" x="67.6275" y="17.78" size="1.27" layer="25" rot="R90"/>
+<attribute name="VALUE" x="71.4375" y="17.78" size="1.27" layer="27" rot="R90"/>
+</element>
+<element name="U2" library="my-power" package="SOT89" value="HT7333" x="30.1625" y="17.145" smashed="yes">
+<attribute name="NAME" x="27.644" y="16.1895" size="0.4064" layer="25" rot="R90"/>
+<attribute name="VALUE" x="33.153" y="16.0155" size="0.4064" layer="27" rot="R90"/>
+</element>
 </elements>
 <signals>
@@
 <wire x1="19.685" y1="14.27793125" x2="19.685" y2="6.6675" width="0.3048" layer="16"/>
 <via x="19.685" y="17.145" extent="1-16" drill="0.6" diameter="1.016"/>
-<wire x1="19.685" y1="14.27793125" x2="19.685" y2="17.145" width="0.3048" layer="16"/>
+<wire x1="19.685" y1="14.31" x2="19.685" y2="17.145" width="0.3048" layer="16"/>
 <wire x1="39.37" y1="11.43" x2="39.21125" y2="11.58875" width="0.3048" layer="16"/>
 <wire x1="20.59" y1="19.84375" x2="20.59" y2="18.05" width="0.3048" layer="1"/>
@@
 <wire x1="14.5575" y1="19.84375" x2="14.5575" y2="18.145" width="0.3048" layer="1"/>
 <wire x1="14.5575" y1="19.84375" x2="11.00125" y2="19.84375" width="0.3048" layer="1"/>
-<contactref element="U1" pad="B+"/>
-<contactref element="BATT1" pad="+"/>
-<wire x1="7.415" y1="14.31" x2="3.605" y2="10.5" width="0.4064" layer="1"/>
-<wire x1="24.935" y1="14.31" x2="7.415" y2="14.31" width="0.4064" layer="1"/>
-<wire x1="24.935" y1="14.31" x2="19.685" y2="14.31" width="0.3048" layer="16"/>
 <wire x1="19.685" y1="14.31" x2="19.685" y2="14.27793125" width="0.3048" layer="16"/>
 </signal>
@@
 <wire x1="50.8" y1="5.08" x2="54.9275" y2="5.08" width="0.3048" layer="16"/>
 </signal>
+<signal name="+BATT">
+<contactref element="U1" pad="B+"/>
+<contactref element="BATT1" pad="+"/>
+<wire x1="7.415" y1="14.31" x2="3.605" y2="10.5" width="0.4064" layer="1"/>
+<wire x1="24.935" y1="14.31" x2="7.415" y2="14.31" width="0.4064" layer="1"/>
+</signal>
 </signals>
+<mfgpreviewcolors>
+<mfgpreviewcolor name="soldermaskcolor" color="0xC8008000"/>
+<mfgpreviewcolor name="silkscreencolor" color="0xFFFEFEFE"/>
+<mfgpreviewcolor name="backgroundcolor" color="0xFF282828"/>
+<mfgpreviewcolor name="coppercolor" color="0xFFFFBF00"/>
+<mfgpreviewcolor name="substratecolor" color="0xFF786E46"/>
+</mfgpreviewcolors>
 </board>
 </drawing>
