File: eagle/MySLipo_v2.0.sch (EAGLE design)
At the start: 23 parts, among them IC1 ATMEGA328, U1 USB_CHARGER, U2 HT7333, U3 ATSHA204A

Commit message: v2.0
Parts:
- removed 18500: SINGLE_BATTERY_HOLDER18650, moje:SINGLE_BATTERY_HOLDER18650
- removed J$1: ANTENNATINY, WeMos-Lora:ANTENNATINY
- removed JP1: (no value), pinhead:PINHD-1X7
- removed R3, R4: 4K7, rcl:R-EU_R0805
- removed R7: 10K, rcl:R-EU_R0805
- removed RFM69W: RADIO_RFM69W_MIN_PAD, mysensors:RADIO_RFM69W_MIN_PAD
- added BATT1: LI-PO_18650, moje:SINGLE_BATTERY_HOLDER18650
- added C5, C6: 100n, rcl:C-EUC0805
- added LED1: yellow, mysensors:LED
- added R10, R11: 10K, rcl:R-EU_R0805
- added R12: 1K2, rcl:R-EU_R0805
- added R8, R9: 1M, rcl:R-EU_R0805
- added S1, S2: MEDER, moje:MEDER
- R5: value 120K -> 1M
- R6: value 220K -> 330K
- U2: device moje:HT73XX -> my-power:HT7333
Connections:
- net N$5 renamed CE
- removed net A0: IC1.PC0(ADC0), JP1.1, R7.1
- removed net A1: IC1.PC1(ADC1), JP1.2
- removed net ANT: J$1.SIGNAL, RFM69W.ANT
- removed net N$6: IC1.PB2(SS/OC1B), NRF24L01+LNA+PA.CSN, NRF24L01.CSN, RFM69W.NSS
- removed net N$8: 18500.+, U1.B+
- removed net SCL: IC1.PC5(ADC5/SCL), JP1.4, R4.1
- removed net SDA: IC1.PC4(ADC4/SDA), JP1.3, R3.1
- new net CSN: IC1.PB2(SS/OC1B), NRF24L01+LNA+PA.CSN, NRF24L01.CSN
- new net D3: IC1.PD3(INT1), R11.1
- new net D7: IC1.PD7(AIN1), LED1.A
- new net N$17: LED1.C, R12.2
- new net N$2: C5.1, R10.2, R9.2, S1.1
- new net N$3: C6.2, R11.2, R8.1, S2.1
- net +3V3: now also C5.2, C6.1, R8.2, R9.1, U2.OUT; no longer JP1.7, R3.2, R4.2, RFM69W.3V3, U2.VOUT
- net D2: now also IC1.PD2(INT0), R10.1; no longer IC1.PD3(INT1), JP1.5
- net GND: now also R12.1, S1.2, S2.2; no longer J$1.GND@0, J$1.GND@1, J$1.GND@2, J$1.GND@3, JP1.6, R7.2, RFM69W.GND, RFM69W.GND1
- net MISO: no longer RFM69W.MISO
- net MOSI: no longer RFM69W.MOSI
- net N$1: no longer IC1.PD2(INT0), RFM69W.DIO0
- net N$9: now also BATT1.-; no longer 18500.-
- net SCK: no longer RFM69W.SCK
- net VBATT: now also BATT1.+, U1.B+
- net VCC: now also U2.IN; no longer U2.VIN
Other:
- moved on the sheet: C1, C2, C3, C4, DS18B20, IC1, NRF24L01, NRF24L01+LNA+PA, PROG, R1, R2, R5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

Commit message: eagle update
Connections:
- new net +BATT: BATT1.+, U1.B+
- net VBATT: no longer BATT1.+, U1.B+
